Commit message: feat(navigation): add basic lidar support

File: apps/ros2/src/raros_navigation/description/core.xacro (robot description, xacro)
@@ -1,5 +1,4 @@
 <?xml version="1.0"?>
 <robot xmlns:xacro="http://www.ros.org/wiki/xacro">
-  <xacro:include filename="inertial_macros.xacro"/>
   <material name="white">
     <color rgba="1 1 1 1"/>
@@ -13,4 +12,7 @@
   <material name="black">
     <color rgba="0 0 0 1"/>
+  </material>
+  <material name="red">
+    <color rgba="1 0 0 1"/>
   </material>
   <!-- BASE LINK -->
@@ -37,75 +39,7 @@
       </geometry>
     </collision>
-    <xacro:inertial_box mass="0.5" x="0.3" y="0.3" z="0.15">
-      <origin xyz="0.15 0 0.075" rpy="0 0 0"/>
-    </xacro:inertial_box>
   </link>
-  <!-- LEFT WHEEL LINK -->
-  <joint name="left_wheel_joint" type="continuous">
-    <parent link="base_link"/>
-    <child link="left_wheel"/>
-    <origin xyz="0 0.175 0" rpy="-${pi/2} 0 0"/>
-    <axis xyz="0 0 1"/>
-  </joint>
-  <link name="left_wheel">
-    <visual>
-      <geometry>
-        <cylinder radius="0.05" length="0.04"/>
-      </geometry>
-      <material name="blue"/>
-    </visual>
-    <collision>
-      <geometry>
-        <cylinder radius="0.05" length="0.04"/>
-      </geometry>
-    </collision>
-    <xacro:inertial_cylinder mass="0.1" length="0.04" radius="0.05">
-      <origin xyz="0 0 0" rpy="0 0 0"/>
-    </xacro:inertial_cylinder>
-  </link>
-  <!-- RIGHT WHEEL LINK -->
-  <joint name="right_wheel_joint" type="continuous">
-    <parent link="base_link"/>
-    <child link="right_wheel"/>
-    <origin xyz="0 -0.175 0" rpy="${pi/2} 0 0"/>
-    <axis xyz="0 0 -1"/>
-  </joint>
-  <link name="right_wheel">
-    <visual>
-      <geometry>
-        <cylinder radius="0.05" length="0.04"/>
-      </geometry>
-      <material name="blue"/>
-    </visual>
-    <collision>
-      <geometry>
-        <cylinder radius="0.05" length="0.04"/>
-      </geometry>
-    </collision>
-    <xacro:inertial_cylinder mass="0.1" length="0.04" radius="0.05">
-      <origin xyz="0 0 0" rpy="0 0 0"/>
-    </xacro:inertial_cylinder>
-  </link>
-  <!-- CASTER WHEEL LINK -->
-  <joint name="caster_wheel_joint" type="fixed">
-    <parent link="chassis"/>
-    <child link="caster_wheel"/>
-    <origin xyz="0.24 0 0"/>
-  </joint>
-  <link name="caster_wheel">
-    <visual>
-      <geometry>
-        <sphere radius="0.05"/>
-      </geometry>
-      <material name="black"/>
-    </visual>
-    <collision>
-      <geometry>
-        <sphere radius="0.05"/>
-      </geometry>
-    </collision>
-    <xacro:inertial_sphere mass="0.1" radius="0.05">
-      <origin xyz="0 0 0" rpy="0 0 0"/>
-    </xacro:inertial_sphere>
-  </link>
+  <gazebo reference="chassis">
+    <material>Gazebo/White</material>
+  </gazebo>
 </robot>

File: apps/ros2/src/raros_navigation/description/robot.urdf.xacro (robot description, xacro)
@@ -2,3 +2,4 @@
 <robot xmlns:xacro="http://www.ros.org/wiki/xacro" name="raros_bot">
   <xacro:include filename="core.xacro"/>
+  <xacro:include filename="lidar.xacro" />
 </robot>

Commit message: feat(urdf): add wheels

File: apps/ros2/src/raros_navigation/description/core.xacro (robot description, xacro)
@@ -1,45 +1,43 @@
-<?xml version="1.0"?>
+<?xml version="1.0" encoding="UTF-8"?>
 <robot xmlns:xacro="http://www.ros.org/wiki/xacro">
-  <material name="white">
-    <color rgba="1 1 1 1"/>
-  </material>
-  <material name="orange">
-    <color rgba="1 0.3 0.1 1"/>
-  </material>
-  <material name="blue">
-    <color rgba="0.2 0.2 1 1"/>
-  </material>
-  <material name="black">
-    <color rgba="0 0 0 1"/>
-  </material>
-  <material name="red">
-    <color rgba="1 0 0 1"/>
-  </material>
-  <!-- BASE LINK -->
-  <link name="base_link">
+  <!-- Define robot constants -->
+  <xacro:property name="base_width" value="0.185"/>
+  <xacro:property name="base_length" value="0.350"/>
+  <xacro:property name="base_height" value="0.04"/>
+  <xacro:property name="wheel_radius" value="0.0420"/>
+  <xacro:property name="wheel_width" value="0.025"/>
+  <xacro:property name="wheel_ygap" value="0.005"/>
+  <xacro:property name="wheel_zoff" value="0.035"/>
+  <xacro:property name="wheel_xoff" value="0.10"/>
+  <xacro:property name="caster_yoff" value="0.05"/>
+  <xacro:property name="caster_xoff" value="0.2"/>
+  <!-- Robot Base -->
+  <link name="base_link"/>
+  <!-- Robot Footprint -->
+  <link name="base_footprint"/>
+  <joint name="base_joint" type="fixed">
+    <parent link="base_link"/>
+    <child link="base_footprint"/>
+    <origin xyz="0.0 0.0 ${-(wheel_radius+wheel_zoff)}" rpy="0 0 0"/>
+  </joint>
+  <!-- Chassis-->
+  <link name="chassis_base">
+    <visual>
+      <geometry>
+        <box size="${base_length} ${base_width} ${base_height}"/>
+      </geometry>
+      <material name="cyan"/>
+    </visual>
   </link>
-  <!-- CHASSIS LINK -->
   <joint name="chassis_joint" type="fixed">
     <parent link="base_link"/>
-    <child link="chassis"/>
-    <origin xyz="-0.1 0 0"/>
+    <child link="chassis_base"/>
+    <origin xyz="${wheel_xoff} 0 0"/>
   </joint>
-  <link name="chassis">
-    <visual>
-      <origin xyz="0.15 0 0.075"/>
-      <geometry>
-        <box size="0.3 0.3 0.15"/>
-      </geometry>
-      <material name="white"/>
-    </visual>
-    <collision>
-      <origin xyz="0.15 0 0.075"/>
-      <geometry>
-        <box size="0.3 0.3 0.15"/>
-      </geometry>
-    </collision>
-  </link>
-  <gazebo reference="chassis">
-    <material>Gazebo/White</material>
-  </gazebo>
+  <!-- Wheels -->
+  <xacro:wheel prefix="drive_wheel_l" y_reflect="1"/>
+  <xacro:wheel prefix="drive_wheel_r" y_reflect="-1"/>
+  <!--  Caster Wheels-->
+  <xacro:caster_wheel prefix="front_caster" y_reflect="1"/>
+  <xacro:caster_wheel prefix="rear_caster" y_reflect="-1"/>
 </robot>

File: apps/ros2/src/raros_navigation/description/lidar.xacro (robot description, xacro)
@@ -1,6 +1,6 @@
-<?xml version="1.0"?>
+<?xml version="1.0" encoding="UTF-8"?>
 <robot xmlns:xacro="http://www.ros.org/wiki/xacro">
   <joint name="laser_joint" type="fixed">
-    <parent link="chassis"/>
+    <parent link="base_link"/>
     <child link="laser_frame"/>
     <origin xyz="0.1 0 0.175" rpy="0 0 0"/>

File: apps/ros2/src/raros_navigation/description/robot.urdf.xacro (robot description, xacro)
@@ -1,5 +1,7 @@
-<?xml version="1.0"?>
-<robot xmlns:xacro="http://www.ros.org/wiki/xacro" name="raros_bot">
+<?xml version="1.0" encoding="UTF-8"?>
+<robot name="raros_bot" xmlns:xacro="http://www.ros.org/wiki/xacro">
+  <xacro:include filename="materials.xacro"/>
+  <xacro:include filename="wheel.xacro"/>
   <xacro:include filename="core.xacro"/>
-  <xacro:include filename="lidar.xacro" />
+  <xacro:include filename="lidar.xacro"/>
 </robot>

Commit message: feat(urdf): update lidar model

File: apps/ros2/src/raros_navigation/description/core.xacro (robot description, xacro)
@@ -3,6 +3,9 @@
   <!-- Define robot constants -->
   <xacro:property name="base_width" value="0.185"/>
-  <xacro:property name="base_length" value="0.350"/>
+  <xacro:property name="base_length" value="0.31"/>
   <xacro:property name="base_height" value="0.04"/>
+  <xacro:property name="top_width" value="0.13"/>
+  <xacro:property name="top_height" value="0.07"/>
+  <xacro:property name="top_length" value="0.23"/>
   <xacro:property name="wheel_radius" value="0.0420"/>
   <xacro:property name="wheel_width" value="0.025"/>
@@ -35,8 +38,22 @@
     <origin xyz="${wheel_xoff} 0 0"/>
   </joint>
+  <!-- Top Chassis-->
+  <link name="chassis_top">
+    <visual>
+      <geometry>
+        <box size="${top_length} ${top_width} ${top_height}"/>
+      </geometry>
+      <material name="cyan"/>
+    </visual>
+  </link>
+  <joint name="top_joint" type="fixed">
+    <parent link="chassis_base"/>
+    <child link="chassis_top"/>
+    <origin xyz="${top_length / 2 - base_length / 2} 0 ${base_height / 2 + top_height / 2}" rpy="0 0 0"/>
+  </joint>
   <!-- Wheels -->
   <xacro:wheel prefix="drive_wheel_l" y_reflect="1"/>
   <xacro:wheel prefix="drive_wheel_r" y_reflect="-1"/>
-  <!--  Caster Wheels-->
+  <!-- Caster Wheels-->
   <xacro:caster_wheel prefix="front_caster" y_reflect="1"/>
   <xacro:caster_wheel prefix="rear_caster" y_reflect="-1"/>

File: apps/ros2/src/raros_navigation/description/lidar.xacro (robot description, xacro)
@@ -1,21 +1,36 @@
 <?xml version="1.0" encoding="UTF-8"?>
 <robot xmlns:xacro="http://www.ros.org/wiki/xacro">
-  <joint name="laser_joint" type="fixed">
-    <parent link="base_link"/>
-    <child link="laser_frame"/>
-    <origin xyz="0.1 0 0.175" rpy="0 0 0"/>
+  <xacro:property name="mount_width" value="0.06"/>
+  <xacro:property name="mount_height" value="0.07"/>
+  <xacro:property name="mount_length" value="0.09"/>
+  <xacro:property name="laser_height" value="0.025"/>
+  <xacro:property name="laser_radius" value="0.035"/>
+  <!-- LIDAR Mount -->
+  <link name="laser_mount">
+    <visual>
+      <geometry>
+        <box size="${mount_length} ${mount_width} ${mount_height}"/>
+      </geometry>
+      <material name="white"/>
+    </visual>
+  </link>
+  <joint name="laser_mount_joint" type="fixed">
+    <parent link="chassis_top"/>
+    <child link="laser_mount"/>
+    <origin xyz="${-mount_width} 0 ${top_height / 2 + mount_height / 2}" rpy="0 0 0"/>
   </joint>
+  <!-- LIDAR Sensor-->
   <link name="laser_frame">
     <visual>
       <geometry>
-        <cylinder radius="0.05" length="0.04"/>
+        <cylinder radius="${laser_radius}" length="${laser_height}"/>
       </geometry>
-      <material name="red"/>
+      <material name="orange"/>
     </visual>
-    <collision>
-      <geometry>
-        <cylinder radius="0.05" length="0.04"/>
-      </geometry>
-    </collision>
   </link>
+  <joint name="laser_joint" type="fixed">
+    <parent link="laser_mount"/>
+    <child link="laser_frame"/>
+    <origin xyz="0 0 ${ mount_height / 2 + laser_height / 2}" rpy="0 0 0"/>
+  </joint>
 </robot>

Commit message: feat(urdf): add collision and inertia properties

File: apps/ros2/src/raros_navigation/description/core.xacro (robot description, xacro)
@@ -32,4 +32,10 @@
       <material name="cyan"/>
     </visual>
+    <collision>
+      <geometry>
+        <box size="${base_length} ${base_width} ${base_height}"/>
+      </geometry>
+    </collision>
+    <xacro:box_inertia m="2" w="${base_width}" d="${base_length}" h="${base_height}"/>
   </link>
   <joint name="chassis_joint" type="fixed">
@@ -46,4 +52,10 @@
       <material name="cyan"/>
     </visual>
+     <collision>
+      <geometry>
+        <box size="${top_length} ${top_width} ${top_height}"/>
+      </geometry>
+    </collision>
+    <xacro:box_inertia m="0.2" w="${top_width}" d="${top_length}" h="${top_height}"/>
   </link>
   <joint name="top_joint" type="fixed">

File: apps/ros2/src/raros_navigation/description/lidar.xacro (robot description, xacro)
@@ -14,4 +14,10 @@
       <material name="white"/>
     </visual>
+    <collision>
+      <geometry>
+        <box size="${mount_length} ${mount_width} ${mount_height}"/>
+      </geometry>
+    </collision>
+    <xacro:box_inertia m="0.1" w="${mount_width}" d="${mount_length}" h="${mount_height}"/>
   </link>
   <joint name="laser_mount_joint" type="fixed">
@@ -28,4 +34,10 @@
       <material name="orange"/>
     </visual>
+      <collision>
+      <geometry>
+        <cylinder radius="${laser_radius}" length="${laser_height}"/>
+      </geometry>
+    </collision>
+    <xacro:cylinder_inertia m="0.5" r="${laser_radius}" h="${laser_height}"/>
   </link>
   <joint name="laser_joint" type="fixed">

File: apps/ros2/src/raros_navigation/description/robot.urdf.xacro (robot description, xacro)
@@ -2,4 +2,5 @@
 <robot name="raros_bot" xmlns:xacro="http://www.ros.org/wiki/xacro">
   <xacro:include filename="materials.xacro"/>
+  <xacro:include filename="inertial_macros.xacro"/>
   <xacro:include filename="wheel.xacro"/>
   <xacro:include filename="core.xacro"/>

File: apps/ros2/src/raros_navigation/description/wheel.xacro (robot description, xacro)
@@ -10,4 +10,11 @@
         <material name="gray"/>
       </visual>
+       <collision>
+        <origin xyz="0 0 0" rpy="${pi/2} 0 0"/>
+        <geometry>
+          <cylinder radius="${wheel_radius}" length="${wheel_width}"/>
+        </geometry>
+      </collision>
+      <xacro:cylinder_inertia m="0.5" r="${wheel_radius}" h="${wheel_width}"/>
     </link>
     <joint name="${prefix}_joint" type="continuous">
@@ -26,4 +33,11 @@
         <material name="gray"/>
       </visual>
+      <collision>
+      <origin xyz="0 0 0" rpy="0 0 0"/>
+      <geometry>
+         <sphere radius="${wheel_radius}"/>
+      </geometry>
+    </collision>
+    <xacro:sphere_inertia m="0.3" r="${wheel_radius}"/>
     </link>
     <joint name="${prefix}_joint" type="fixed">
