Commit message: feat(navigation): add gazebo simulation

File: apps/ros2/src/raros_navigation/description/lidar.xacro (robot description, xacro)
@@ -34,5 +34,5 @@
       <material name="orange"/>
     </visual>
-      <collision>
+    <collision>
       <geometry>
         <cylinder radius="${laser_radius}" length="${laser_height}"/>
@@ -46,3 +46,31 @@
     <origin xyz="0 0 ${ mount_height / 2 + laser_height / 2}" rpy="0 0 0"/>
   </joint>
+  <gazebo reference="laser_frame">
+    <material>Gazebo/Red</material>
+    <sensor name="laser" type="ray">
+      <pose>0 0 0 0 0 0</pose>
+      <visualize>true</visualize>
+      <update_rate>10</update_rate>
+      <ray>
+        <scan>
+          <horizontal>
+            <samples>360</samples>
+            <min_angle>-3.14</min_angle>
+            <max_angle>3.14</max_angle>
+          </horizontal>
+        </scan>
+        <range>
+          <min>0.3</min>
+          <max>12</max>
+        </range>
+      </ray>
+      <plugin name="laser_controller" filename="libgazebo_ros_ray_sensor.so">
+        <ros>
+          <argument>~/out:=scan</argument>
+        </ros>
+        <output_type>sensor_msgs/LaserScan</output_type>
+        <frame_name>laser_frame</frame_name>
+      </plugin>
+    </sensor>
+  </gazebo>
 </robot>

File: apps/ros2/src/raros_navigation/description/robot.urdf.xacro (robot description, xacro)
@@ -3,4 +3,5 @@
   <xacro:include filename="materials.xacro"/>
   <xacro:include filename="inertial_macros.xacro"/>
+  <xacro:include filename="gazebo_control.xacro"/>
   <xacro:include filename="wheel.xacro"/>
   <xacro:include filename="core.xacro"/>

File: apps/ros2/src/raros_navigation/description/wheel.xacro (robot description, xacro)
@@ -10,5 +10,5 @@
         <material name="gray"/>
       </visual>
-       <collision>
+      <collision>
         <origin xyz="0 0 0" rpy="${pi/2} 0 0"/>
         <geometry>
@@ -24,4 +24,7 @@
       <axis xyz="0 1 0"/>
     </joint>
+    <gazebo reference="${prefix}_link">
+      <material>Gazebo/Gray</material>
+    </gazebo>
   </xacro:macro>
   <xacro:macro name="caster_wheel" params="prefix y_reflect">
@@ -34,10 +37,10 @@
       </visual>
       <collision>
-      <origin xyz="0 0 0" rpy="0 0 0"/>
-      <geometry>
-         <sphere radius="${wheel_radius}"/>
-      </geometry>
-    </collision>
-    <xacro:sphere_inertia m="0.3" r="${wheel_radius}"/>
+        <origin xyz="0 0 0" rpy="0 0 0"/>
+        <geometry>
+          <sphere radius="${wheel_radius}"/>
+        </geometry>
+      </collision>
+      <xacro:sphere_inertia m="0.3" r="${wheel_radius}"/>
     </link>
     <joint name="${prefix}_joint" type="fixed">
@@ -46,4 +49,9 @@
       <origin xyz="${caster_xoff} ${y_reflect*caster_yoff} ${-wheel_zoff}" rpy="0 0 0"/>
     </joint>
+    <gazebo reference="${prefix}_link">
+      <material>Gazebo/Black</material>
+      <mu1 value="0.001"/>
+      <mu2 value="0.001"/>
+    </gazebo>
   </xacro:macro>
 </robot>
